Commit message: Rvis Poppy

File: poppy_torso_description/urdf/poppy_torso.urdf (robot description, URDF)
Before this commit: robot poppy_torso, 17 links, 16 joints
Joints:
- joint bust_x: limit lower=-1.57079 upper=1.57079 effort=10 velocity=3.1415 -> lower=-1.0 upper=1.0 effort=10 velocity=3.1415
- joint bust_y: limit lower=-1.57079 upper=1.57079 effort=10 velocity=3.1415 -> lower=-1.0 upper=0.44 effort=10 velocity=3.1415
- joint head_y: limit lower=-1.57079 upper=1.57079 effort=10 velocity=3.1415 -> lower=-0.74 upper=0.2 effort=10 velocity=3.1415
- joint head_z: limit lower=-1.57079 upper=1.57079 effort=10 velocity=3.1415 -> lower=-1.0 upper=1.0 effort=10 velocity=3.1415
- joint l_elbow_y: limit lower=-1.57079 upper=1.57079 effort=10 velocity=3.1415 -> lower=-2.4 upper=0.0 effort=10 velocity=3.1415
- joint l_shoulder_x: limit lower=-1.57079 upper=1.57079 effort=10 velocity=3.1415 -> lower=-0.4 upper=1.8 effort=10 velocity=3.1415
- joint l_shoulder_y: limit lower=-1.57079 upper=1.57079 effort=10 velocity=3.1415 -> lower=-1.8 upper=0.3 effort=10 velocity=3.1415
- joint r_elbow_y: limit lower=-1.57079 upper=1.57079 effort=10 velocity=3.1415 -> lower=0.0 upper=2.4 effort=10 velocity=3.1415
- joint r_shoulder_x: limit lower=-1.57079 upper=1.57079 effort=10 velocity=3.1415 -> lower=-0.4 upper=1.8 effort=10 velocity=3.1415
- joint r_shoulder_y: limit lower=-1.57079 upper=1.57079 effort=10 velocity=3.1415 -> lower=-0.3 upper=1.8 effort=10 velocity=3.1415

Commit message: MoveIt! working with 1 planning group

File: poppy_torso_description/urdf/poppy_torso.urdf (robot description, URDF)
Before this commit: robot poppy_torso, 17 links, 16 joints
Joints:
- joint l_shoulder_y: limit lower=-1.8 upper=0.3 effort=10 velocity=3.1415 -> lower=-1.8 upper=1.7 effort=10 velocity=3.1415
- joint r_shoulder_y: limit lower=-0.3 upper=1.8 effort=10 velocity=3.1415 -> lower=-1.7 upper=1.8 effort=10 velocity=3.1415
